File: boards/PIG-19/PIG-19.kicad_sch (KiCad schematic)
At the start: 9 parts

Commit message: V1 of PCB
Parts:
- removed C2: 0.1uF, Capacitor_SMD:C_0805_2012Metric, symbol Device:C
- removed R4: 10k, Resistor_SMD:R_0805_2012Metric, symbol Device:R_US
- removed SW2: ~, customFootprints:rockerSwitch-434133025816, symbol custom:rockerSwitch
- added SW4: ~, customFootprints:rockerSwitch-434133025816, symbol custom:rockerSwitch
- C3: value 1uF -> 0.1uF; footprint Capacitor_SMD:C_0805_2012Metric -> Capacitor_SMD:C_0603_1608Metric; MANUFACTURER 581-KAF21KR71E105KU -> 581-KAM21KR72A104KU
- C4: footprint Capacitor_SMD:C_0805_2012Metric -> Capacitor_SMD:C_0603_1608Metric; MANUFACTURER 581-KAF21KR72A104KL -> 581-CM105X5R226M16AT
- C5: footprint Capacitor_SMD:C_0805_2012Metric -> Capacitor_SMD:C_0603_1608Metric; MANUFACTURER 581-KAM21KR72A104KU -> 581-KAF15AR71H104KM
- R3: value 10k -> 1k; footprint Resistor_SMD:R_0805_2012Metric -> Resistor_SMD:R_0603_1608Metric; MANUFACTURER 667-ERA-6APB103V -> 652-CRT0805AFY-1001E
Connections:
- net 3_mot is gone; now on net INT1: MCU1.33 (IO37)
- net 4_mot is gone; now on net SDA: MCU1.34 (IO38)
- net Boot is gone; now on an unnamed net: MCU1.4 (IO0)
- net +3V3: now also R3.2; no longer R3.1
- net GND: now also SW4.2
- net INT1: no longer MCU1.36 (IO40)
- net INT2: now also MCU1.36 (IO40); no longer MCU1.35 (IO39)
- net SCL: now also MCU1.35 (IO39); no longer MCU1.32 (IO36)
- net SDA: no longer MCU1.31 (IO35)
- net mot-1: now also MCU1.37 (IO41)
- net mot-2: now also MCU1.9 (IO5)
- net LED_S2: now reaches MCU1.38 (IO42)
- net LED_S1: now reaches MCU1.41 (IO45)
- net Trig_2: now reaches MCU1.5 (IO1)
- net Trig_1: now reaches MCU1.6 (IO2)
- net Echo_2: now reaches MCU1.7 (IO3)
- net Echo_1: now reaches MCU1.8 (IO4)
- net 1_mot: no longer names the net of MCU1.14 (IO10)
- net 2_mot: no longer names the net of MCU1.15 (IO11)
- net EN: no longer names the net of C3.2, MCU1.45 (EN)
- net EN: now also R3.1, SW4.1; no longer R3.2
- new net Batt_S: MCU1.32 (IO36)
- no-connect marks 26 -> 20
Other:
- sheet ESP32-CAM renamed sensors
- sheet BLDC Motors ports: added none; removed mot-3, mot-4
- sheet Battery Sensing Circuit ports: added Batt_Sense; removed none
- sheet Directional&Large Leds ports: added LED_S1, LED_S2; removed none
- sheet IMU ports: added INT1, INT2, SCL, SDA; removed none
- sheet sensors ports: added Echo_1, Echo_2, Trig_1, Trig_2; removed none
- note removed: "Attach battery sensing circuit"
- note removed: "Boot Button"
- note removed: "EN Button"
