File: boards/PIG-19/PIG-19.kicad_sch (KiCad schematic)
At the start: 7 parts

Commit message: I2C pull up resistors
Changed lines of the file:
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@@
 	(text_box "Additional Items to outline on Board \n- USB-HUB \n- 196-DEVBOARD "
 		(exclude_from_sim no)
-		(at 156.21 25.4 0)
+		(at 154.94 19.05 0)
 		(size 26.67 17.78)
 		(stroke
@@
 	)
 	(sheet
-		(at 156.21 46.99)
+		(at 196.85 27.94)
 		(size 34.29 11.43)
 		(fields_autoplaced yes)
@@
 		)
 		(property "Sheetname" "Mounting"
-			(at 156.21 46.2784 0)
+			(at 196.85 27.2284 0)
 			(effects
 				(font
@@
 		)
 		(property "Sheetfile" "mounting.kicad_sch"
-			(at 156.21 59.0046 0)
-			(effects
-				(font
+			(at 196.85 39.9546 0)
+			(effects
+				(font

Commit message: commit for adin to review
Connections:
- net INT3: now reaches MCU1.10 (IO6)
- no-connect marks 20 -> 19
Other:
- sheet IMU ports: added INT3; removed none
Changed lines of the file:
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@@
-	)
-	(no_connect
-		(at 85.09 69.85)
 	)
 	(no_connect
@@
 	(wire
 		(pts
+			(xy 242.57 90.17) (xy 237.49 90.17)
+		)
+		(stroke
+			(width 0)
+			(type default)
+		)
+	)
+	(wire
+		(pts
 			(xy 128.27 40.64) (xy 128.27 41.91)
 		)
@@
 		(pts
 			(xy 115.57 57.15) (xy 128.27 57.15)
+		)
+		(stroke
+			(width 0)
+			(type default)
+		)
+	)
+	(wire
+		(pts
+			(xy 76.2 69.85) (xy 85.09 69.85)
 		)
 		(stroke
@@
 		)
 	)
+	(label "INT3"
+		(at 237.49 90.17 0)
+		(fields_autoplaced yes)
+		(effects
+			(font
+				(size 1.27 1.27)
+			)
+			(justify left bottom)
+		)
+	)
 	(label "Batt_S"
 		(at 125.73 72.39 180)
@@
 	(label "DP"
 		(at 238.76 54.61 0)
+		(fields_autoplaced yes)
+		(effects
+			(font
+				(size 1.27 1.27)
+			)
+			(justify left bottom)
+		)
+	)
+	(label "INT3"
+		(at 76.2 69.85 0)
 		(fields_autoplaced yes)
 		(effects
@@
 			)
 		)
+		(pin "INT3" input
+			(at 242.57 90.17 180)
+			(effects
+				(font
+					(size 1.27 1.27)
+				)
+				(justify left)
+			)
+		)
 		(instances
 			(project "PIG-19"
@@
 	)
 	(sheet
-		(at 196.85 27.94)
+		(at 43.18 152.4)
 		(size 34.29 11.43)
 		(fields_autoplaced yes)
@@
 		)
 		(property "Sheetname" "Mounting"
-			(at 196.85 27.2284 0)
+			(at 43.18 151.6884 0)
 			(effects
 				(font
@@
 		)
 		(property "Sheetfile" "mounting.kicad_sch"
-			(at 196.85 39.9546 0)
-			(effects
-				(font
+			(at 43.18 164.4146 0)
+			(effects
+				(font

Commit message: board updates
Connections:
- net ENB: now reaches MCU1.16 (IO12)
- net IN4: now reaches MCU1.17 (IO13)
- net IN3: now reaches MCU1.18 (IO14)
- net IN2: now reaches MCU1.19 (IO15)
- net IN1: now reaches MCU1.20 (IO16)
- net ENA: now reaches MCU1.21 (IO17)
- no-connect marks 19 -> 13
Other:
- sheet BLDC Motors renamed MOTORS
- sheet MOTORS ports: added ENA, ENB, IN1, IN2, IN3, IN4; removed none

Commit message: Final Board Revision - pls order this one TAs
Changed lines of the file:
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@@
 	(wire
 		(pts
-			(xy 85.09 69.85) (xy 80.01 69.85)
+			(xy 85.09 69.85) (xy 76.2 69.85)
 		)
 		(stroke
@@
 	)
 	(label "INT3"
-		(at 80.01 69.85 0)
+		(at 76.2 69.85 0)
 		(fields_autoplaced yes)
 		(effects

Commit message: this bom file to order pls
Parts:
- SW1, SW4: now left out of the parts list
Changed lines of the file:
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@@
 		(unit 1)
 		(exclude_from_sim no)
-		(in_bom yes)
+		(in_bom no)
 		(on_board yes)
 		(dnp no)
@@
 		(unit 1)
 		(exclude_from_sim no)
-		(in_bom yes)
+		(in_bom no)
 		(on_board yes)
 		(dnp no)
