File: boards/PIG-19/batterysensor.kicad_sch (KiCad schematic)
At the start: 0 parts

Commit message: V1 of PCB
Parts:
- added R8: 470k, Resistor_SMD:R_0603_1608Metric, symbol Device:R_US
- added R9: 530k, Resistor_SMD:R_0603_1608Metric, symbol Device:R_US
Connections:
- new net +BATT: R8.1
- new net Batt_Sense: R8.2, R9.1
- new net GND: R9.2
Other:
- note removed: "MAX17043"
