File: boards/PIG-19/power.kicad_sch (KiCad schematic)
At the start: 15 parts, among them J10 Conn_01x02_Pin, J11 USB4105-GF-A, J9 XT30PW-M, Q1 PMOS, SW3 SW_Nidec_CAS-120A1

Commit message: V1 of PCB
Parts:
- removed J10: Conn_01x02_Pin, Connector_PinHeader_2.54mm:PinHeader_1x02_P2.54mm_Horizontal, symbol Connector:Conn_01x02_Pin
- C1, C6: footprint Capacitor_SMD:C_0805_2012Metric -> Capacitor_SMD:C_0603_1608Metric
- R1, R2, R5, R6: footprint Resistor_SMD:R_0805_2012Metric -> Resistor_SMD:R_0603_1608Metric
- SW3: footprint Button_Switch_SMD:SW_DPDT_CK_JS202011JCQN -> JS102011JAQN:SW_JS102011JAQN
