File: boards/PIG-19/power.kicad_sch (KiCad schematic)
At the start: 14 parts, among them J11 USB4105-GF-A, J9 XT30PW-M, Q1 PMOS, SW3 SW_Nidec_CAS-120A1

Commit message: Final Board Revision - pls order this one TAs
Parts:
- added TP1, TP2: TestPoint, TestPoint:TestPoint_Pad_D2.0mm, symbol Connector:TestPoint
- R2: value 500k -> 20k; MANUFACTURER ERJ-2RKF4993X -> 5-2176074-3
Connections:
- net DN: now also TP2.1
- net DP: now also TP1.1
- net PWR-DIODE: now reaches C1.1, D2.1 (K), D3.1 (K), LDO1.5 (EN), LDO1.8 (IN)
Other:
- note added: "Swap 500k Resistor -> 20k resistor"

Commit message: Added BOM for main board
Parts:
- TP1, TP2: now left out of the parts list
Changed lines of the file:
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@@
 		(unit 1)
 		(exclude_from_sim no)
-		(in_bom yes)
+		(in_bom no)
 		(on_board yes)
 		(dnp no)
@@
 		(unit 1)
 		(exclude_from_sim no)
-		(in_bom yes)
-		(on_board yes)
-		(dnp no)
+		(in_bom no)
+		(on_board yes)
+		(dnp no)
