File: boards/PIG-19/PIG-19.kicad_pcb (KiCad board)
At the start: 2 copper layers, 70 x 40 mm, 40 parts, among them J1 XT30PW-F, J11 USB4105-GF-A, J2 XT30PW-F, J5 Conn_01x02_Pin, J6 Conn_01x02_Pin, J9 XT30PW-M, Q1 PMOS, SW3 SW_Nidec_CAS-120A1, U1 LM2940S-5.0

Commit message: commit for adin to review
Parts:
- added BNO1: Conn_01x05_Pin, Connector_PinHeader_2.54mm:PinHeader_1x05_P2.54mm_Vertical, F.Cu at (146.6, 54.8)
- added R10: 10k, Resistor_SMD:R_0603_1608Metric, F.Cu at (144.7, 57.4)
- added R4: 10k, Resistor_SMD:R_0603_1608Metric, F.Cu at (144.8, 59.0)
- moved C6 0.72 mm to (148.8, 64.3)
- moved C7 0.24 mm to (182.5, 56.0)
- moved R7 0.09 mm to (179.5, 52.8)
Connections:
- MCU1 pad 10: unconnected-(MCU1-IO6-Pad10) -> /INT3
Routing:
- net /SCL: track 11.1 -> 72.0 mm, vias 0 -> 1
- net /SDA: track 11.5 -> 51.4 mm, vias 0 -> 1
- net /INT3: track 0.00 -> 17.5 mm, vias 0 -> 2
- net +3V3: track 123.9 -> 138.8 mm, vias 8 -> 10
- net +BATT: track 99.2 -> 95.9 mm
- net +V_USB: track 58.4 -> 55.6 mm
- net /mot-2: track 23.4 -> 25.8 mm, vias 0 -> 1
- net GND: track 15.9 -> 13.6 mm, vias 29 -> 33
- net /Echo_1: track 21.1 -> 20.5 mm
- net +5V: track 84.5 -> 85.0 mm, vias 3 -> 5
Other:
- board text added: "3V3"

Commit message: board updates
Parts:
- added RescueDCPin1: Conn_01x06_Pin, Connector_PinHeader_2.54mm:PinHeader_1x06_P2.54mm_Vertical, F.Cu at (166.4, 81.5)
- R1: value 510 -> 100
- R8: value 470k -> 1M
- R9: value 530k -> 500k
- moved R1 18.5 mm to (168.5, 86.7)
- moved H2 18.5 mm to (129.5, 95.6)
- moved H3 18.4 mm to (190.5, 95.5)
- moved Q1 18.3 mm to (152.9, 90.7)
- moved J9 18.3 mm to (142.1, 97.9)
- moved R5 18.3 mm to (168.9, 90.9)
- moved R6 18.3 mm to (162.4, 90.9)
- moved U1 18.3 mm to (177.1, 90.6)
- moved D1 18.3 mm to (168.6, 88.4)
- moved R2 18.3 mm to (157.8, 90.5)
- moved J11 18.3 mm to (165.1, 98.1)
- moved SW3 18.3 mm to (154.6, 97.1)
- moved R10 13.1 mm to (142.3, 70.3)
- moved R9 13.1 mm to (183.0, 71.3)
- moved C3 13.1 mm to (173.6, 56.9)
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Connections:
- MCU1 pad 16: unconnected-(MCU1-IO12-Pad16) -> /ENB
- MCU1 pad 17: unconnected-(MCU1-IO13-Pad17) -> /IN4
- MCU1 pad 18: unconnected-(MCU1-IO14-Pad18) -> /IN3
- MCU1 pad 19: unconnected-(MCU1-IO15-Pad19) -> /IN2
- MCU1 pad 20: unconnected-(MCU1-IO16-Pad20) -> /IN1
- MCU1 pad 21: unconnected-(MCU1-IO17-Pad21) -> /ENA
- R1 pad 1: +3V3 -> +5V
Routing:
- net /ENA: track 0.00 -> 14.4 mm
- net /DN: track 19.9 -> 32.6 mm
- net /IN1: track 0.00 -> 12.6 mm
- net +3V3: track 138.8 -> 126.3 mm, vias 10 -> 9
- net +BATT: track 95.9 -> 108.1 mm, vias 8 -> 5
- net +5V: track 85.0 -> 96.5 mm
- net /DP: track 20.6 -> 31.9 mm
- net /IN2: track 0.00 -> 10.9 mm
- net /IN3: track 0.00 -> 9.40 mm
- net /IN4: track 0.00 -> 7.36 mm
- net /ENB: track 0.00 -> 6.45 mm
- net +V_USB: track 55.6 -> 60.6 mm
- net GND: vias 33 -> 39
Other:
- board size 70 x 40 mm -> 70.1 x 45.4 mm
- board text added: "PWR"

Commit message: Final Board Revision - pls order this one TAs
Parts:
- added LM298NPWR1: Conn_01x02_Pin, Connector_PinHeader_2.54mm:PinHeader_1x02_P2.54mm_Vertical, F.Cu at (188.8, 88.2)
- added TP1: TestPoint, TestPoint:TestPoint_Pad_D2.0mm, F.Cu at (157.4, 85.2)
- added TP2: TestPoint, TestPoint:TestPoint_Pad_D2.0mm, F.Cu at (161.5, 85.2)
- R2: value 500k -> 20k
- moved D2 0.13 mm to (138.3, 76.0)
- moved D3 0.12 mm to (138.2, 78.8)
Connections:
- C1 pad 1: Net-(D2-K) -> PWR-DIODE
- C2 pad 1: +BATT -> PWR-DIODE
- D2 pad 1: Net-(D2-K) -> PWR-DIODE
- D3 pad 1: Net-(D2-K) -> PWR-DIODE
- LDO1 pad 5: Net-(D2-K) -> PWR-DIODE
- LDO1 pad 8: Net-(D2-K) -> PWR-DIODE
- U1 pad 1: +BATT -> PWR-DIODE
Routing:
- net +BATT: track 108.1 -> 4.78 mm, vias 5 -> 11
- net +5V: track 96.5 -> 0.00 mm, vias 5 -> 6
- net +V_USB: track 60.6 -> 7.46 mm, vias 2 -> 6
- net /DP: track 31.9 -> 42.0 mm, vias 0 -> 2
- net GND: track 13.6 -> 7.47 mm, vias 39 -> 90
- net +3V3: track 126.3 -> 120.8 mm, vias 9 -> 10
- net /DN: track 32.6 -> 35.5 mm
- net /mot-1: track 28.0 -> 25.6 mm
- net /LED_S2: track 24.2 -> 22.2 mm
- net /Echo_2: track 21.8 -> 20.3 mm
- net /INT2: track 13.8 -> 12.5 mm
- net /Trig_1: track 16.7 -> 15.3 mm
- net /Trig_2: track 18.1 -> 16.8 mm
- net /Echo_1: track 20.5 -> 19.3 mm
- net /SDA: track 51.4 -> 50.3 mm
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- added copper zone on F.Cu, net +3V3
- added copper zone on In1.Cu, net +5V
- added copper zone on In1.Cu, net +BATT
- added copper zone on In1.Cu, net +V_USB
- added copper zone on In2.Cu, net GND
- added copper zone on F.Cu, net PWR-DIODE
- removed copper zone on F.Cu, net Net-(D2-K)
Other:
- copper layers 2 -> 4
- board text added: "BATT|GND"
- board text added: "USB"

Commit message: Order & Check TAs pls ty ty
Routing:
- net GND: track 7.47 -> 24.3 mm, vias 90 -> 107
- net PWR-DIODE: vias 5 -> 6
- net +3V3: vias 10 -> 9
- added copper zone on B.Cu, net PWR-DIODE
- removed copper zone on B.Cu, net GND
