File: boards/uSlime_BNO085_Module/BNO085.kicad_sch (KiCad schematic)
At the start: 14 parts, among them J1 Conn_01x05, U1 BNO085

Commit message: other PIG-19 & BNO Board pls, ty
Parts:
- R3, R4: value 2.2k -> 4.7k
Changed lines of the file:
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@@
 			)
 		)
-		(property "Value" "2.2k"
+		(property "Value" "4.7k"
 			(at 190.5 78.7399 0)
 			(effects
@@
 			)
 		)
-		(property "Value" "2.2k"
+		(property "Value" "4.7k"
 			(at 181.61 77.4699 0)
 			(effects

Commit message: update bno BOM
Parts:
- C1, C2, C3, C4: MANUFACTURER (none) -> KAF15AR71H104KM
- J1: now left out of the parts list
- R1, R2, R5: MANUFACTURER (none) -> RN73C1J10KBTD
- R3, R4: MANUFACTURER (none) -> TNPU06034K70AYEN00
- R6, R7: MANUFACTURER (none) -> CPF0603B2K2E1
- U1: MANUFACTURER (none) -> BNO085
